File: elec/layout/default/solar-charger.kicad_pcb (KiCad board)
At the start: 2 copper layers, 225.7 x 100.8 mm, 4 parts

Commit message: design v3
Parts:
- added C1: Multilayer Ceramic Capacitors MLCC - SMD/SMT 4.7uF 16V 0805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, lib:C0805, F.Cu at (156.0, 50.4)
- added C2: Multilayer Ceramic Capacitors MLCC - SMD/SMT 100nF 10V 0402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, lib:C0402, F.Cu at (154.3, 51.5)
- added R1: 100mW Thick Film Resistors ±100ppm/℃ ±1% 5.1MΩ 0603 Chip Re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, lib:R0603, F.Cu at (153.1, 58.2)
- added R10: 62.5mW Thick Film Resistors ±100ppm/℃ ±1% 4.02MΩ 0402 Chip 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, lib:R0402, F.Cu at (151.0, 54.5)
- added R2: 62.5mW Thick Film Resistors ±100ppm/℃ ±1% 4.87MΩ 0402 Chip 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, lib:R0402, F.Cu at (150.8, 57.4)
- added R3: 250mW Thick Film Resistors 200V ±100ppm/℃ ±1% -55℃~+155℃ 4.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, lib:R1206, F.Cu at (159.3, 54.9)
- added R4: 62.5mW Thick Film Resistors ±100ppm/℃ ±1% 4.87MΩ 0402 Chip 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, lib:R0402, F.Cu at (159.3, 57.3)
- added R5: 250mW Thick Film Resistors ±100ppm/℃ ±1% 715kΩ 1206 Chip Re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, lib:R1206, F.Cu at (156.4, 58.3)
- added R6: 62.5mW ±1% ±400ppm/℃ 4.99MΩ 0402 Chip Resistor - Surface Mo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, lib:R0402, F.Cu at (158.5, 60.7)
- added R7: 62.5mW ±1% ±400ppm/℃ 4.99MΩ 0402 Chip Resistor - Surface Mo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, lib:R0402, F.Cu at (156.0, 60.7)
- added R8: 62.5mW Thick Film Resistors ±100ppm/℃ ±1% 6.04MΩ 0402 Chip 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, lib:R0402, F.Cu at (161.4, 57.0)
- added R9: 100mW Thick Film Resistors ±100ppm/℃ ±1% 10MΩ 0603 Chip Res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, lib:R0603, F.Cu at (161.0, 59.5)
- added U5: , lib:CONN-SMD_P2.00_S2B-PH-SM4-TB-LF-SN, F.Cu at (157.8, 42.9)
- added U6: , lib:CONN-SMD_P2.00_S2B-PH-SM4-TB-LF-SN, F.Cu at (143.5, 61.0)
- moved U2 98.8 mm to (147.8, 42.5)
- moved U1 94.9 mm to (154.5, 54.6)
- moved U4 94.2 mm to (143.5, 52.2)
- moved U3 93.2 mm to (150.0, 51.3)
Connections:
- net AVSS renamed avss
- net EP renamed ep
- net LBST renamed lbst
- net OT_PROG renamed ot_prog
- net VBAT_OK renamed vbat_ok
- net VREF_SAMP renamed vref_samp
- net _2 renamed gnd
- U1 pad 1: VSS -> vss
- U1 pad 10: OK_PROG -> ok_prog
- U1 pad 13: VSS -> vss2
- U1 pad 14: VBAT -> vbat
- U1 pad 15: VSTOR -> vcc
- U1 pad 3: VOC_SAMP -> voc_samp
- U1 pad 6: VBAT_OV -> vbat_ov
- U1 pad 7: VRDIV -> vrdiv
- U1 pad 8: VBAT_UV -> vbat_uv
- U1 pad 9: OK_HYST -> ok_hyst
Routing:
- net gnd: track 0.00 -> 52.8 mm, vias 0 -> 4
- net vcc: track 0.00 -> 23.8 mm, vias 0 -> 2
- net _1: track 0.00 -> 20.7 mm
- net voc_samp: track 0.00 -> 15.2 mm, vias 0 -> 2
- net lbst: track 0.00 -> 11.3 mm
- net vbat: track 0.00 -> 10.1 mm
- net vrdiv: track 0.00 -> 6.68 mm
- net vbat_uv: track 0.00 -> 6.62 mm
- net ok_hyst: track 0.00 -> 5.58 mm
- net vbat_ov: track 0.00 -> 5.50 mm
- net ok_prog: track 0.00 -> 4.43 mm
- net p2: track 0.00 -> 2.02 mm
- added copper zone on B.Cu, net gnd
Other:
- board size 225.7 x 100.8 mm -> 25 x 27.4 mm
- board text added: "+"
- board text added: "Vbattery"
- board text added: "Vload"
- board text added: "Vsolar"
